File: Hardware/Pro-Mini-Candy.brd (EAGLE design)
At the start: 17.8 x 33 mm, 29 parts, among them Q1 8/16/20MHz, U1 ATMEGA328, U2 MIC5205

Commit message: Updating Silk
Parts:
- moved U$2 4.02 mm to (13.1, 3.94)
- moved U$3 2.51 mm to (12.2, 2.26), turned to 0 degrees
